Commit message: Update bumperbot.urdf.xacro

File: bumperbot_description/urdf/bumperbot.urdf.xacro (robot description, xacro)
@@ -165,3 +165,27 @@
         <child link="imu_link" />
     </joint>
+    <link name="laser_link">
+        <inertial>
+            <origin xyz="-0.011945780406062 -0.000381929217680526 -0.0170649378129477" rpy="0 0 0" />
+            <mass value="0.073084435549317" />
+            <inertia ixx="1.96074931730795E-05" ixy="-3.62091076640009E-07" ixz="4.28230084046735E-07" iyy="2.40983835136327E-05" iyz="1.50180909250652E-08" izz="4.14184164228595E-05" />
+        </inertial>
+        <visual>
+            <origin xyz="0 0 0" rpy="0 0 0" />
+            <geometry>
+                <mesh filename="package://bumperbot_description/meshes/laser_link.STL" />
+            </geometry>
+        </visual>
+        <collision>
+            <origin xyz="0 0 0" rpy="0 0 0" />
+            <geometry>
+                <mesh filename="package://bumperbot_description/meshes/laser_link.STL" />
+            </geometry>
+        </collision>
+    </link>
+    <joint name="laser_joint" type="fixed">
+        <origin xyz="0.0 0.0 0.1208" rpy="0 0 3.14" />
+        <parent link="base_link" />
+        <child link="laser_link" />
+    </joint>
 </robot>
